File: Lasgun.sch (KiCad schematic (older format))
At the start: 23 parts, among them CON1 AVR-ISP-6, IC1 ATMEGA328P-A, M1 STM32F042G6, M2 EPSON_FA-20H_CRYSTAL, P1 CONN_01X03, P2 CONN_01X03, Q1 Q_NMOS_GSD

Commit message: Added voltage reg
Parts:
- added VREG1: VREG_5PINS-SOT-23-5, james:James-SOT23-5, symbol VREG_5PINS-SOT-23-5
- added regc1: 10uf, Capacitors_SMD:C_1206_HandSoldering, symbol C
- BATSIG1: footprint (none) -> Pin_Headers:Pin_Header_Straight_1x02
- CON1: footprint AVR-ISP-6 -> Pin_Headers:Pin_Header_Straight_2x03
Connections:
- net +3V3: now also VREG1.5 (OUT)
- net +BATT: now also VREG1.1 (IN), VREG1.3 (EN), regc1.1
- net GND: now also VREG1.2 (GND), regc1.2
Other:
- note added: "POWER"
- note added: "PROG HEADER"
Changed lines of the file:
@@
 LED_FET
 $Comp
-L +3.3V #PWR12
+L +3.3V #PWR01
 U 1 1 5637E45F
 P 5150 2950
-F 0 "#PWR12" H 5150 2800 50  0001 C CNN
+F 0 "#PWR01" H 5150 2800 50  0001 C CNN
 F 1 "+3.3V" H 5150 3090 50  0000 C CNN
 F 2 "" H 5150 2950 60  0000 C CNN
@@
 $EndComp
 $Comp
-L +3.3V #PWR9
+L +3.3V #PWR02
 U 1 1 5637E47B
 P 3050 2950
-F 0 "#PWR9" H 3050 2800 50  0001 C CNN
+F 0 "#PWR02" H 3050 2800 50  0001 C CNN
 F 1 "+3.3V" H 3050 3090 50  0000 C CNN
 F 2 "" H 3050 2950 60  0000 C CNN
@@
 $EndComp
 $Comp
-L +3.3V #PWR8
+L +3.3V #PWR03
 U 1 1 5637E4EB
 P 3000 4100
-F 0 "#PWR8" H 3000 3950 50  0001 C CNN
+F 0 "#PWR03" H 3000 3950 50  0001 C CNN
 F 1 "+3.3V" H 3000 4240 50  0000 C CNN
 F 2 "" H 3000 4100 60  0000 C CNN
@@
 $EndComp
 $Comp
-L GND #PWR6
+L GND #PWR04
 U 1 1 5637E5A9
 P 2950 6600
-F 0 "#PWR6" H 2950 6350 50  0001 C CNN
+F 0 "#PWR04" H 2950 6350 50  0001 C CNN
 F 1 "GND" H 2950 6450 50  0000 C CNN
 F 2 "" H 2950 6600 60  0000 C CNN
@@
 $EndComp
 $Comp
-L GND #PWR13
+L GND #PWR05
 U 1 1 5637E6C2
 P 5150 3100
-F 0 "#PWR13" H 5150 2850 50  0001 C CNN
+F 0 "#PWR05" H 5150 2850 50  0001 C CNN
 F 1 "GND" H 5150 2950 50  0000 C CNN
 F 2 "" H 5150 3100 60  0000 C CNN
@@
 $EndComp
 $Comp
-L GND #PWR3
+L GND #PWR06
 U 1 1 5637EAF7
 P 1900 2550
-F 0 "#PWR3" H 1900 2300 50  0001 C CNN
+F 0 "#PWR06" H 1900 2300 50  0001 C CNN
 F 1 "GND" H 1900 2400 50  0000 C CNN
 F 2 "" H 1900 2550 60  0000 C CNN
@@
 $EndComp
 $Comp
-L +3.3V #PWR16
+L +3.3V #PWR07
 U 1 1 5637EC9B
 P 5850 5100
-F 0 "#PWR16" H 5850 4950 50  0001 C CNN
+F 0 "#PWR07" H 5850 4950 50  0001 C CNN
 F 1 "+3.3V" H 5850 5240 50  0000 C CNN
 F 2 "" H 5850 5100 60  0000 C CNN
@@
 $EndComp
 $Comp
-L GND #PWR4
+L GND #PWR08
 U 1 1 56380212
 P 2250 5650
-F 0 "#PWR4" H 2250 5400 50  0001 C CNN
+F 0 "#PWR08" H 2250 5400 50  0001 C CNN
 F 1 "GND" H 2250 5500 50  0000 C CNN
 F 2 "" H 2250 5650 60  0000 C CNN
@@
 $EndComp
 $Comp
-L GND #PWR18
+L GND #PWR09
 U 1 1 56380940
 P 8050 5200
-F 0 "#PWR18" H 8050 4950 50  0001 C CNN
+F 0 "#PWR09" H 8050 4950 50  0001 C CNN
 F 1 "GND" H 8050 5050 50  0000 C CNN
 F 2 "" H 8050 5200 60  0000 C CNN
@@
 $EndComp
 $Comp
-L GND #PWR17
+L GND #PWR010
 U 1 1 5638095C
 P 7050 5750
-F 0 "#PWR17" H 7050 5500 50  0001 C CNN
+F 0 "#PWR010" H 7050 5500 50  0001 C CNN
 F 1 "GND" H 7050 5600 50  0000 C CNN
 F 2 "" H 7050 5750 60  0000 C CNN
@@
 $EndComp
 $Comp
-L GND #PWR20
+L GND #PWR011
 U 1 1 56380B14
 P 9050 2700
-F 0 "#PWR20" H 9050 2450 50  0001 C CNN
+F 0 "#PWR011" H 9050 2450 50  0001 C CNN
 F 1 "GND" H 9050 2550 50  0000 C CNN
 F 2 "" H 9050 2700 60  0000 C CNN
@@
 $EndComp
 $Comp
-L +3.3V #PWR14
+L +3.3V #PWR012
 U 1 1 5638162C
 P 5800 2950
-F 0 "#PWR14" H 5800 2800 50  0001 C CNN
+F 0 "#PWR012" H 5800 2800 50  0001 C CNN
 F 1 "+3.3V" H 5800 3090 50  0000 C CNN
 F 2 "" H 5800 2950 60  0000 C CNN
@@
 $EndComp
 $Comp
-L GND #PWR15
+L GND #PWR013
 U 1 1 56381702
 P 5800 3450
-F 0 "#PWR15" H 5800 3200 50  0001 C CNN
+F 0 "#PWR013" H 5800 3200 50  0001 C CNN
 F 1 "GND" H 5800 3300 50  0000 C CNN
 F 2 "" H 5800 3450 60  0000 C CNN
@@
 IR_RECEIVER1
 $Comp
-L +3.3V #PWR11
+L +3.3V #PWR014
 U 1 1 56382F17
 P 4650 1250
-F 0 "#PWR11" H 4650 1100 50  0001 C CNN
+F 0 "#PWR014" H 4650 1100 50  0001 C CNN
 F 1 "+3.3V" H 4650 1390 50  0000 C CNN
 F 2 "" H 4650 1250 60  0000 C CNN
@@
 $EndComp
 $Comp
-L GND #PWR10
+L GND #PWR015
 U 1 1 56382F30
 P 4500 1250
-F 0 "#PWR10" H 4500 1000 50  0001 C CNN
+F 0 "#PWR015" H 4500 1000 50  0001 C CNN
 F 1 "GND" H 4500 1100 50  0000 C CNN
 F 2 "" H 4500 1250 60  0000 C CNN
@@
 $EndComp
 $Comp
-L +BATT #PWR19
+L +BATT #PWR016
 U 1 1 563957B8
 P 9050 700
-F 0 "#PWR19" H 9050 550 50  0001 C CNN
+F 0 "#PWR016" H 9050 550 50  0001 C CNN
 F 1 "+BATT" H 9050 840 50  0000 C CNN
 F 2 "" H 9050 700 60  0000 C CNN
@@
 F 0 "CON1" H 9545 4640 50  0000 C CNN
 F 1 "AVR-ISP-6" H 9385 4170 50  0000 L BNN
-F 2 "AVR-ISP-6" V 9130 4440 50  0001 C CNN
+F 2 "Pin_Headers:Pin_Header_Straight_2x03" V 9130 4440 50  0001 C CNN
 F 3 "" H 9625 4400 60  0000 C CNN
 	1    9650 4400
@@
 Reuse the AVR connector for programming the STM32\navr_sck = swdclk\navr_miso = swdio
 $Comp
-L +3.3V #PWR23
+L +3.3V #PWR017
 U 1 1 56396A2E
 P 10150 4300
-F 0 "#PWR23" H 10150 4150 50  0001 C CNN
+F 0 "#PWR017" H 10150 4150 50  0001 C CNN
 F 1 "+3.3V" H 10150 4440 50  0000 C CNN
 F 2 "" H 10150 4300 60  0000 C CNN
@@
 $EndComp
 $Comp
-L GND #PWR24
+L GND #PWR018
 U 1 1 56396A46
 P 10150 4600
-F 0 "#PWR24" H 10150 4350 50  0001 C CNN
+F 0 "#PWR018" H 10150 4350 50  0001 C CNN
 F 1 "GND" H 10150 4450 50  0000 C CNN
 F 2 "" H 10150 4600 60  0000 C CNN
@@
 IR_RECEIVER2
 $Comp
-L +3.3V #PWR7
+L +3.3V #PWR019
 U 1 1 563977FA
 P 3000 1250
-F 0 "#PWR7" H 3000 1100 50  0001 C CNN
+F 0 "#PWR019" H 3000 1100 50  0001 C CNN
 F 1 "+3.3V" H 3000 1390 50  0000 C CNN
 F 2 "" H 3000 1250 60  0000 C CNN
@@
 $EndComp
 $Comp
-L GND #PWR5
+L GND #PWR020
 U 1 1 56397800
 P 2850 1250
-F 0 "#PWR5" H 2850 1000 50  0001 C CNN
+F 0 "#PWR020" H 2850 1000 50  0001 C CNN
 F 1 "GND" H 2850 1100 50  0000 C CNN
 F 2 "" H 2850 1250 60  0000 C CNN
@@
 F 0 "BATSIG1" H 9800 5550 50  0000 C CNN
 F 1 "BAT_SIG" V 9900 5350 50  0000 C CNN
-F 2 "" H 9800 5350 60  0000 C CNN
+F 2 "Pin_Headers:Pin_Header_Straight_1x02" H 9800 5350 60  0001 C CNN
 F 3 "" H 9800 5350 60  0000 C CNN
 	1    9800 5350
@@
 $EndComp
 $Comp
-L GND #PWR22
+L GND #PWR021
 U 1 1 5639872B
 P 9350 5500
-F 0 "#PWR22" H 9350 5250 50  0001 C CNN
+F 0 "#PWR021" H 9350 5250 50  0001 C CNN
 F 1 "GND" H 9350 5350 50  0000 C CNN
 F 2 "" H 9350 5500 60  0000 C CNN
@@
 $EndComp
 $Comp
-L +3V3 #PWR21
+L +3V3 #PWR022
 U 1 1 56398753
 P 9350 5350
-F 0 "#PWR21" H 9350 5200 50  0001 C CNN
+F 0 "#PWR022" H 9350 5200 50  0001 C CNN
 F 1 "+3V3" H 9350 5490 50  0000 C CNN
 F 2 "" H 9350 5350 60  0000 C CNN
@@
 MICRO_RXIN
 $Comp
-L +BATT #PWR1
+L +BATT #PWR023
 U 1 1 56399F00
 P 600 750
-F 0 "#PWR1" H 600 600 50  0001 C CNN
+F 0 "#PWR023" H 600 600 50  0001 C CNN
 F 1 "+BATT" H 600 890 50  0000 C CNN
 F 2 "" H 600 750 60  0000 C CNN
@@
 	600  1650 600  1750
 $Comp
-L GND #PWR2
+L GND #PWR024
 U 1 1 5639A2CE
 P 600 1750
-F 0 "#PWR2" H 600 1500 50  0001 C CNN
+F 0 "#PWR024" H 600 1500 50  0001 C CNN
 F 1 "GND" H 600 1600 50  0000 C CNN
 F 2 "" H 600 1750 60  0000 C CNN
@@
 Text Notes 7300 3350 0    39   ~ 0
 TODO: Need to add the PFET to kill off power to the external flight control board
+$Comp
+L VREG_5PINS-SOT-23-5 VREG1
+U 1 1 5639C5BC
+P 1850 4550
+F 0 "VREG1" H 1550 4875 50  0000 L BNN
+F 1 "VREG_5PINS-SOT-23-5" H 1550 4150 50  0000 L BNN
+F 2 "james:James-SOT23-5" H 1880 4700 20  0001 C CNN
+F 3 "" H 1850 4550 60  0000 C CNN
+	1    1850 4550
+	1    0    0    -1
+$EndComp
+$Comp
+L GND #PWR025
+U 1 1 5639C8D0
+P 1000 4850
+F 0 "#PWR025" H 1000 4600 50  0001 C CNN
+F 1 "GND" H 1000 4700 50  0000 C CNN
+F 2 "" H 1000 4850 60  0000 C CNN
+F 3 "" H 1000 4850 60  0000 C CNN
+	1    1000 4850
+	1    0    0    -1
+$EndComp
+$Comp
+L +BATT #PWR026
+U 1 1 5639CA5D
+P 1050 4100
+F 0 "#PWR026" H 1050 3950 50  0001 C CNN
+F 1 "+BATT" H 1050 4240 50  0000 C CNN
+F 2 "" H 1050 4100 60  0000 C CNN
+F 3 "" H 1050 4100 60  0000 C CNN
+	1    1050 4100
+	1    0    0    -1
+$EndComp
+$Comp
+L +3.3V #PWR027
+U 1 1 5639CA7A
+P 2600 4250
+F 0 "#PWR027" H 2600 4100 50  0001 C CNN
+F 1 "+3.3V" H 2600 4390 50  0000 C CNN
+F 2 "" H 2600 4250 60  0000 C CNN
+F 3 "" H 2600 4250 60  0000 C CNN
+	1    2600 4250
+	1    0    0    -1
+$EndComp
+Wire Wire Line
+	700  4350 1350 4350
+Wire Wire Line
+	1050 4350 1050 4100
+Wire Wire Line
+	1000 4550 1350 4550
+Wire Wire Line
+	1350 4750 1200 4750
+Wire Wire Line
+	1200 4750 1200 4350
+Connection ~ 1200 4350
+Wire Wire Line
+	2350 4350 2600 4350
+Wire Wire Line
+	2600 4350 2600 4250
+$Comp
+L C regc1
+U 1 1 5639D6EF
+P 700 4600
+F 0 "regc1" H 725 4700 50  0000 L CNN
+F 1 "10uf" H 725 4500 50  0000 L CNN
+F 2 "Capacitors_SMD:C_1206_HandSoldering" H 738 4450 30  0001 C CNN
+F 3 "" H 700 4600 60  0000 C CNN
+	1    700  4600
+	1    0    0    -1
+$EndComp
+Wire Wire Line
+	1000 4550 1000 4850
+Wire Wire Line
+	700  4750 700  4800
+Wire Wire Line
+	700  4800 1000 4800
+Connection ~ 1000 4800
+Wire Wire Line
+	700  4350 700  4450
+Connection ~ 1050 4350
+Text Notes 1700 4050 0    118  ~ 0
+POWER
+Text Notes 8950 3950 0    118  ~ 0
+PROG HEADER
 $EndSCHEMATC

Commit message: routing
Parts:
- removed M2: EPSON_FA-20H_CRYSTAL, Ava:Ava-EPSON-FA-20H-CRYSTAL, symbol EPSON_FA-20H_CRYSTAL
- removed VREG1: VREG_5PINS-SOT-23-5, james:James-SOT23-5, symbol VREG_5PINS-SOT-23-5
- removed cy1, cy2: 8pf, Capacitors_SMD:C_0603, symbol C
- added D3: LED, LEDs:LED-3MM, symbol LED
- added VREG1: VREG_3PINS-SOT-223, dp_devices:dp_devices-SOT-23, symbol VREG_3PINS-SOT-223
- BATSIG1: footprint Pin_Headers:Pin_Header_Straight_1x02 -> Socket_Strips:Socket_Strip_Angled_1x03
- C1, C2, C3: footprint Capacitors_SMD:C_0603 -> Capacitors_SMD:C_0603_HandSoldering
- R1, R2, R3, R4, R5, R6: footprint Resistors_SMD:R_0603 -> Resistors_SMD:R_0603_HandSoldering
- regc1: footprint Capacitors_SMD:C_1206_HandSoldering -> Capacitors_SMD:C_1206
Connections:
- net labels removed: +3V3
Other:
- note added: "IR DETECTORS"
- note added: "MCP1700T-3302E/TT"
- note removed: "IR DETECTOR"
Changed lines of the file:
@@
 F 0 "R1" V 2780 2550 50  0000 C CNN
 F 1 "10k" V 2700 2550 50  0000 C CNN
-F 2 "Resistors_SMD:R_0603" V 2630 2550 30  0001 C CNN
+F 2 "Resistors_SMD:R_0603_HandSoldering" V 2630 2550 30  0001 C CNN
 F 3 "" H 2700 2550 30  0000 C CNN
 	1    2700 2550
@@
 F 0 "R3" V 5930 5350 50  0000 C CNN
 F 1 "10K" V 5850 5350 50  0000 C CNN
-F 2 "Resistors_SMD:R_0603" V 5780 5350 30  0001 C CNN
+F 2 "Resistors_SMD:R_0603_HandSoldering" V 5780 5350 30  0001 C CNN
 F 3 "" H 5850 5350 30  0000 C CNN
 	1    5850 5350
@@
 BAT_MON
 $Comp
-L EPSON_FA-20H_CRYSTAL M2
-U 1 1 5637FD73
-P 7300 5000
-F 0 "M2" H 7400 5040 50  0000 L BNN
-F 1 "EPSON_FA-20H_CRYSTAL" H 7400 4900 50  0000 L BNN
-F 2 "Ava:Ava-EPSON-FA-20H-CRYSTAL" H 7330 5150 20  0001 C CNN
-F 3 "" H 7300 5000 60  0000 C CNN
-	1    7300 5000
-	0    -1   -1   0
-$EndComp
-$Comp
 L C C1
 U 1 1 5637FF63
@@
 F 0 "C1" H 3075 5050 50  0000 L CNN
 F 1 "100nf" H 3075 4850 50  0000 L CNN
-F 2 "Capacitors_SMD:C_0603" H 3088 4800 30  0001 C CNN
+F 2 "Capacitors_SMD:C_0603_HandSoldering" H 3088 4800 30  0001 C CNN
 F 3 "" H 3050 4950 60  0000 C CNN
 	1    3050 4950
@@
 F 0 "C2" H 3275 5050 50  0000 L CNN
 F 1 "100nf" H 3275 4850 50  0000 L CNN
-F 2 "Capacitors_SMD:C_0603" H 3288 4800 30  0001 C CNN
+F 2 "Capacitors_SMD:C_0603_HandSoldering" H 3288 4800 30  0001 C CNN
 F 3 "" H 3250 4950 60  0000 C CNN
 	1    3250 4950
@@
 732-FA20H-16F12Z-AC3\nSmall and cheap crystal.\n
 $Comp
-L C cy1
-U 1 1 5638066C
-P 7050 5500
-F 0 "cy1" H 7075 5600 50  0000 L CNN
-F 1 "8pf" H 7075 5400 50  0000 L CNN
-F 2 "Capacitors_SMD:C_0603" H 7088 5350 30  0001 C CNN
-F 3 "" H 7050 5500 60  0000 C CNN
-	1    7050 5500
-	1    0    0    -1
-$EndComp
-$Comp
-L C cy2
-U 1 1 563806D2
-P 8050 4950
-F 0 "cy2" H 8075 5050 50  0000 L CNN
-F 1 "8pf" H 8075 4850 50  0000 L CNN
-F 2 "Capacitors_SMD:C_0603" H 8088 4800 30  0001 C CNN
-F 3 "" H 8050 4950 60  0000 C CNN
-	1    8050 4950
-	1    0    0    -1
-$EndComp
-$Comp
 L GND #PWR09
 U 1 1 56380940
@@
 F 0 "C3" H 5825 3250 50  0000 L CNN
 F 1 "100nf" H 5825 3050 50  0000 L CNN
-F 2 "Capacitors_SMD:C_0603" H 5838 3000 30  0001 C CNN
+F 2 "Capacitors_SMD:C_0603_HandSoldering" H 5838 3000 30  0001 C CNN
 F 3 "" H 5800 3150 60  0000 C CNN
 	1    5800 3150
@@
 F 0 "R4" V 8630 2500 50  0000 C CNN
 F 1 "10K" V 8550 2500 50  0000 C CNN
-F 2 "Resistors_SMD:R_0603" V 8480 2500 30  0001 C CNN
+F 2 "Resistors_SMD:R_0603_HandSoldering" V 8480 2500 30  0001 C CNN
 F 3 "" H 8550 2500 30  0000 C CNN
 	1    8550 2500
@@
 MICROCONTROLLER\nSTM32 OR ATMEGA328
 Text Notes 3650 1600 0    118  ~ 0
-IR DETECTOR
+IR DETECTORS
 Wire Wire Line
 	3350 2550 2850 2550
@@
 F 0 "R6" V 8230 2300 50  0000 C CNN
 F 1 "100" V 8150 2300 50  0000 C CNN
-F 2 "Resistors_SMD:R_0603" V 8080 2300 30  0001 C CNN
+F 2 "Resistors_SMD:R_0603_HandSoldering" V 8080 2300 30  0001 C CNN
 F 3 "" H 8150 2300 30  0000 C CNN
 	1    8150 2300
@@
 F 0 "BATSIG1" H 9800 5550 50  0000 C CNN
 F 1 "BAT_SIG" V 9900 5350 50  0000 C CNN
-F 2 "Pin_Headers:Pin_Header_Straight_1x02" H 9800 5350 60  0001 C CNN
+F 2 "Socket_Strips:Socket_Strip_Angled_1x03" H 9800 5350 60  0001 C CNN
 F 3 "" H 9800 5350 60  0000 C CNN
 	1    9800 5350
@@
 F 3 "" H 9350 5500 60  0000 C CNN
 	1    9350 5500
-	1    0    0    -1
-$EndComp
-$Comp
-L +3V3 #PWR022
-U 1 1 56398753
-P 9350 5350
-F 0 "#PWR022" H 9350 5200 50  0001 C CNN
-F 1 "+3V3" H 9350 5490 50  0000 C CNN
-F 2 "" H 9350 5350 60  0000 C CNN
-F 3 "" H 9350 5350 60  0000 C CNN
-	1    9350 5350
 	1    0    0    -1
 $EndComp
@@
 MICRO_RXIN
 $Comp
-L +BATT #PWR023
+L +BATT #PWR022
 U 1 1 56399F00
 P 600 750
-F 0 "#PWR023" H 600 600 50  0001 C CNN
+F 0 "#PWR022" H 600 600 50  0001 C CNN
 F 1 "+BATT" H 600 890 50  0000 C CNN
 F 2 "" H 600 750 60  0000 C CNN
@@
 F 0 "R2" V 680 1050 50  0000 C CNN
 F 1 "10k" V 600 1050 50  0000 C CNN
-F 2 "Resistors_SMD:R_0603" V 530 1050 30  0001 C CNN
+F 2 "Resistors_SMD:R_0603_HandSoldering" V 530 1050 30  0001 C CNN
 F 3 "" H 600 1050 30  0000 C CNN
 	1    600  1050
@@
 F 0 "R5" V 680 1500 50  0000 C CNN
 F 1 "1k" V 600 1500 50  0000 C CNN
-F 2 "Resistors_SMD:R_0603" V 530 1500 30  0001 C CNN
+F 2 "Resistors_SMD:R_0603_HandSoldering" V 530 1500 30  0001 C CNN
 F 3 "" H 600 1500 30  0000 C CNN
 	1    600  1500
@@
 	600  1650 600  1750
 $Comp
-L GND #PWR024
+L GND #PWR023
 U 1 1 5639A2CE
 P 600 1750
-F 0 "#PWR024" H 600 1500 50  0001 C CNN
+F 0 "#PWR023" H 600 1500 50  0001 C CNN
 F 1 "GND" H 600 1600 50  0000 C CNN
 F 2 "" H 600 1750 60  0000 C CNN
@@
 TODO: Need to add the PFET to kill off power to the external flight control board
 $Comp
-L VREG_5PINS-SOT-23-5 VREG1
-U 1 1 5639C5BC
-P 1850 4550
-F 0 "VREG1" H 1550 4875 50  0000 L BNN
-F 1 "VREG_5PINS-SOT-23-5" H 1550 4150 50  0000 L BNN
-F 2 "james:James-SOT23-5" H 1880 4700 20  0001 C CNN
-F 3 "" H 1850 4550 60  0000 C CNN
-	1    1850 4550
-	1    0    0    -1
-$EndComp
-$Comp
-L GND #PWR025
+L GND #PWR024
 U 1 1 5639C8D0
 P 1000 4850
-F 0 "#PWR025" H 1000 4600 50  0001 C CNN
+F 0 "#PWR024" H 1000 4600 50  0001 C CNN
 F 1 "GND" H 1000 4700 50  0000 C CNN
 F 2 "" H 1000 4850 60  0000 C CNN
@@
 $EndComp
 $Comp
-L +BATT #PWR026
+L +BATT #PWR025
 U 1 1 5639CA5D
 P 1050 4100
-F 0 "#PWR026" H 1050 3950 50  0001 C CNN
+F 0 "#PWR025" H 1050 3950 50  0001 C CNN
 F 1 "+BATT" H 1050 4240 50  0000 C CNN
 F 2 "" H 1050 4100 60  0000 C CNN
@@
 $EndComp
 $Comp
-L +3.3V #PWR027
+L +3.3V #PWR026
 U 1 1 5639CA7A
 P 2600 4250
-F 0 "#PWR027" H 2600 4100 50  0001 C CNN
+F 0 "#PWR026" H 2600 4100 50  0001 C CNN
 F 1 "+3.3V" H 2600 4390 50  0000 C CNN
 F 2 "" H 2600 4250 60  0000 C CNN
@@
 $EndComp
 Wire Wire Line
-	700  4350 1350 4350
+	700  4350 1500 4350
 Wire Wire Line
 	1050 4350 1050 4100
-Wire Wire Line
-	1000 4550 1350 4550
-Wire Wire Line
-	1350 4750 1200 4750
-Wire Wire Line
-	1200 4750 1200 4350
 Connection ~ 1200 4350
-Wire Wire Line
-	2350 4350 2600 4350
 Wire Wire Line
 	2600 4350 2600 4250
@@
 F 0 "regc1" H 725 4700 50  0000 L CNN
 F 1 "10uf" H 725 4500 50  0000 L CNN
-F 2 "Capacitors_SMD:C_1206_HandSoldering" H 738 4450 30  0001 C CNN
+F 2 "Capacitors_SMD:C_1206" H 738 4450 30  0001 C CNN
 F 3 "" H 700 4600 60  0000 C CNN
 	1    700  4600
 	1    0    0    -1
 $EndComp
-Wire Wire Line
-	1000 4550 1000 4850
 Wire Wire Line
 	700  4750 700  4800
@@
 Text Notes 8950 3950 0    118  ~ 0
 PROG HEADER
+Wire Wire Line
+	5200 6000 5700 6000
+Text GLabel 5700 6000 2    39   Input ~ 0
+IR_RECEIVER2
+Text GLabel 6200 3100 2    39   Input ~ 0
+IR_RECEIVER1
+Text GLabel 6200 3200 2    39   Input ~ 0
+IR_RECEIVER2
+$Comp
+L LED D3
+U 1 1 5639F268
+P 6550 7150
+F 0 "D3" H 6550 7250 50  0000 C CNN
+F 1 "LED" H 6550 7050 50  0000 C CNN
+F 2 "LEDs:LED-3MM" H 6550 7150 60  0001 C CNN
+F 3 "" H 6550 7150 60  0000 C CNN
+	1    6550 7150
+	0    -1   -1   0
+$EndComp
+$Comp
+L +3.3V #PWR027
+U 1 1 5639F2F6
+P 6550 6700
+F 0 "#PWR027" H 6550 6550 50  0001 C CNN
+F 1 "+3.3V" H 6550 6840 50  0000 C CNN
+F 2 "" H 6550 6700 60  0000 C CNN
+F 3 "" H 6550 6700 60  0000 C CNN
+	1    6550 6700
+	1    0    0    -1
+$EndComp
+Wire Wire Line
+	6550 6950 6550 6700
+Text Notes 1500 4700 0    39   ~ 0
+MCP1700T-3302E/TT
+$Comp
+L VREG_3PINS-SOT-223 VREG1
+U 1 1 563A6BBE
+P 1900 4350
+F 0 "VREG1" H 1600 4580 50  0000 L BNN
+F 1 "VREG_3PINS-SOT-223" H 1600 4490 50  0000 L BNN
+F 2 "dp_devices:dp_devices-SOT-23" H 1930 4500 20  0001 C CNN
+F 3 "" H 1900 4350 60  0000 C CNN
+	1    1900 4350
+	1    0    0    -1
+$EndComp
+Wire Wire Line
+	2300 4350 2600 4350
+Wire Wire Line
+	1900 4650 1000 4650
+Connection ~ 1000 4650
+Wire Wire Line
+	1000 4650 1000 4850
+$Comp
+L +BATT #PWR028
+U 1 1 563A89E2
+P 9350 5350
+F 0 "#PWR028" H 9350 5200 50  0001 C CNN
+F 1 "+BATT" H 9350 5490 50  0000 C CNN
+F 2 "" H 9350 5350 60  0000 C CNN
+F 3 "" H 9350 5350 60  0000 C CNN
+	1    9350 5350
+	0    -1   -1   0
+$EndComp
 $EndSCHEMATC
